File: jvc43.sch (KiCad schematic (older format))
At the start: 2 parts, among them X101 25 MHz

Commit message: Forward progress: - Ripped up a good chunk of the old place&route around the PHYs - Swizzled graphical placement of LAN8831 diff pair pins, to make the trace   routing be straight-thru.  This also involved swapping the polarity I'm   feeding into the magnetics.  Bonus: the magnetics-to-RJ45 is now straight,   instead of having to go around the back sides! - Adjusted some default trace spacings because of the tiny 0.4mm QFN:   - Switched default traces from 8mil to 7.8mil   - Switched diff pairs from 8.8/8.1 to 7.4/7.8 - Whoops, not all the 0.1uF decoupling caps were 0402 sized yet - Filled in a lot of specific vendor P/Ns for resistors & capacitors, to make   dealing with assembly houses easier
PHY1 has all its close-in decoupling caps placed & routed, PHY2 does not yet.
Parts:
- added R101, R102, R103, R104, R105, R106, R107, R108, R109, R110, R111: 22, Resistor_SMD:R_0402_1005Metric, symbol Device:R_US
Connections:
- net CLK_W2B: now also R109.1
- net EN_W2B: now also R110.1
- net ER_W2B: now also R111.1
- new net Ethernet1/RXCLK: R109.2
- new net Ethernet1/RXDV: R110.2
- new net Ethernet1/RXER: R111.2
- new net RXD0: R101.2
- new net RXD1: R102.2
- new net RXD2: R103.2
- new net RXD3: R104.2
- new net RXD4: R105.2
- new net RXD5: R106.2
- new net RXD6: R107.2
- new net RXD7: R108.2
- new net TXD0: R101.1
- new net TXD1: R102.1
- new net TXD2: R103.1
- new net TXD3: R104.1
- new net TXD4: R105.1
- new net TXD5: R106.1
- new net TXD6: R107.1
- new net TXD7: R108.1
Other:
- note added: "Place resistors near PHY #1"

Commit message: - Sanitized some of the capacitor voltages / footprints - Selected mfr P/Ns for *all* parts - Placed and routed most of the series resistors, ran into a problem with the   VDD vias on PHY1..... - Placed and routed (all?) the bypass caps for PHY2
Parts:
- C101: value 10n -> 0.1u; footprint Capacitor_SMD:C_0603_1608Metric -> Capacitor_SMD:C_0402_1005Metric; Part# (none) -> CGA2B1X7R1C104K050BC; Voltage 6.3V -> 16V
Changed lines of the file:
@@
 P 1900 3800
 F 0 "C101" H 2015 3846 50  0000 L CNN
-F 1 "10n" H 2015 3755 50  0000 L CNN
-F 2 "Capacitor_SMD:C_0603_1608Metric" H 1938 3650 50  0001 C CNN
+F 1 "0.1u" H 2015 3755 50  0000 L CNN
+F 2 "Capacitor_SMD:C_0402_1005Metric" H 1938 3650 50  0001 C CNN
 F 3 "~" H 1900 3800 50  0001 C CNN
-F 4 "6.3V" H 1900 3800 50  0001 C CNN "Voltage"
+F 4 "16V" H 1900 3800 50  0001 C CNN "Voltage"
+F 5 "CGA2B1X7R1C104K050BC" H 0   0   50  0001 C CNN "Part#"
 	1    1900 3800
 	1    0    0    -1
@@
 Wire Wire Line
 	3500 5500 3500 5400
-Wire Bus Line
-	4300 1100 4300 1800
-Wire Bus Line
-	5700 1100 5700 1800
-Wire Bus Line
-	1600 1100 2800 1100
 $Comp
 L power:+1V1 #PWR0110
@@
 	1    0    0    -1
 $EndComp
+Wire Bus Line
+	4300 1100 4300 1800
+Wire Bus Line
+	5700 1100 5700 1800
+Wire Bus Line
+	1600 1100 2800 1100
 $EndSCHEMATC
