File: psu.sch (KiCad schematic (older format))
At the start: 23 parts, among them J401 USB_C_Receptacle_USB2.0, U401 LTC3622*DE

Commit message: Re-calculated my power budget for the new PHY chips.  It went waaaay down! - The switcher output caps are slight overkill but are okay to stay as-is - The inductors definitely needed to be increased in value
Parts:
- L402: value 4.2uH -> 6.2uH; Part# SRR5028-4R2Y -> SRR5028-6R2Y
- L403: value 6.2uH -> 15uH; Part# SRR5028-6R2Y -> SRR5028-150Y
Changed lines of the file:
@@
 P 8100 2200
 F 0 "L402" V 8200 2200 50  0000 C CNN
-F 1 "4.2uH" V 8050 2200 50  0000 C CNN
+F 1 "6.2uH" V 8050 2200 50  0000 C CNN
 F 2 "myfp:L_5.8x5.8mm_cutcir_6.3mm" H 8100 2200 50  0001 C CNN
 F 3 "~" H 8100 2200 50  0001 C CNN
-F 4 "SRR5028-4R2Y" V 8100 2200 50  0001 C CNN "Part#"
+F 4 "SRR5028-6R2Y" V 8100 2200 50  0001 C CNN "Part#"
 	1    8100 2200
 	0    -1   -1   0
@@
 P 9850 2200
 F 0 "L403" V 9950 2200 50  0000 C CNN
-F 1 "6.2uH" V 9800 2200 50  0000 C CNN
+F 1 "15uH" V 9800 2200 50  0000 C CNN
 F 2 "myfp:L_5.8x5.8mm_cutcir_6.3mm" H 9850 2200 50  0001 C CNN
 F 3 "~" H 9850 2200 50  0001 C CNN
-F 4 "SRR5028-6R2Y" V 9850 2200 50  0001 C CNN "Part#"
+F 4 "SRR5028-150Y" V 9850 2200 50  0001 C CNN "Part#"
 	1    9850 2200
 	0    -1   -1   0
